Commit message: fix(模型): 回填底盘外形与麦轮厚度几何参数
按实测底盘 220×192×145 mm、麦轮厚 30 mm 更新 URDF，并同步
mecanum 运动学 lx+ly=0.206，消除占位几何与实车不一致。

File: src/smartcar_bringup/urdf/smartcar.urdf.xacro (robot description, xacro)
@@ -9,5 +9,5 @@
        track_width    左右轮距（左轮到右轮）[m]
      轮子相对 base_link 的位置 = (±wheelbase/2, ±track_width/2)。
-     注意：几何占位值（wheelbase/track_width）待实车测量后回填，
+     注意：轴距/轮距须与实车测量一致（底盘 220×192×145 mm，麦轮厚 30 mm），
      见 docs/协议总结.md §7 Q7。它们同时决定：
        1) 轮子 link 的摆放（可视化 / TF）
@@ -22,12 +22,15 @@
   <xacro:arg name="serial_port" default="/dev/ttyUSB0"/>
   <xacro:arg name="baud_rate" default="115200"/>
-  <!-- ===== 几何常量（单位 m）===== -->
+  <!-- ===== 几何常量（单位 m，2026-07-20 实车测量回填）===== -->
+  <!-- 底盘外形：长 220 mm × 宽 192 mm × 高 145 mm；麦轮 Ø60 mm、厚 30 mm。
+       轴距/轮距暂按底盘长宽近似（轮心距未单独卷尺时）；改此处时必须同步
+       controllers.yaml 的 sum_of_robot_center_projection_on_X_Y_axis。 -->
   <xacro:property name="wheel_radius" value="0.03"/>   <!-- 麦轮 Ø60mm → r=0.03 -->
-  <xacro:property name="wheel_width" value="0.04"/>    <!-- 轮宽，仅用于可视化 -->
-  <xacro:property name="wheelbase" value="0.20"/>      <!-- 前后轴距（占位，实测替换）-->
-  <xacro:property name="track_width" value="0.20"/>    <!-- 左右轮距（占位，实测替换）-->
-  <xacro:property name="base_length" value="0.24"/>
-  <xacro:property name="base_width" value="0.16"/>
-  <xacro:property name="base_height" value="0.06"/>
+  <xacro:property name="wheel_width" value="0.03"/>    <!-- 轮厚 30 mm，仅可视化 -->
+  <xacro:property name="wheelbase" value="0.220"/>     <!-- 前后轴距 ≈ 底盘长 -->
+  <xacro:property name="track_width" value="0.192"/>   <!-- 左右轮距 ≈ 底盘宽 -->
+  <xacro:property name="base_length" value="0.220"/>
+  <xacro:property name="base_width" value="0.192"/>
+  <xacro:property name="base_height" value="0.145"/>
   <xacro:property name="base_mass" value="2.0"/>
   <xacro:property name="wheel_mass" value="0.15"/>

Commit message: fix(urdf): 修正轮子在底盘 Z 轴正中间而非底部的问题
根因：base_footprint_joint 的 Z 偏移仅设为 wheel_radius（轮子中心高度），但未考虑底盘 box 自身高度，导致底盘 box 几何中心与轮子中心重合，视觉上轮子位于车辆垂直中心且底盘一半埋入地下。

修复：base_footprint_joint origin Z: wheel_radius -> base_height/2 + wheel_radius；轮关节 origin Z: 0 -> -base_height/2

验证：底盘底面位于轮子中心高度(z=0.03)，轮子底部着地(z=0)，底盘完全在地面上方，惯量自洽，运动学参数不受影响。同时删除重复的临时修正文件 smartcar_fixed.urdf.xacro 和 smartcar_fixed.launch.py。

File: src/smartcar_bringup/urdf/smartcar.urdf.xacro (robot description, xacro)
@@ -8,5 +8,6 @@
        wheelbase      前后轮轴距（前轴到后轴）[m]
        track_width    左右轮距（左轮到右轮）[m]
-     轮子相对 base_link 的位置 = (±wheelbase/2, ±track_width/2)。
+     轮子相对 base_link 的位置 = (±wheelbase/2, ±track_width/2, -base_height/2)，
+     Z 偏移使轮子位于底盘底面而非几何中心。
      注意：轴距/轮距须与实车测量一致（底盘 220×192×145 mm，麦轮厚 30 mm），
      见 docs/协议总结.md §7 Q7。它们同时决定：
@@ -68,6 +69,8 @@
     <parent link="base_footprint"/>
     <child link="base_link"/>
-    <!-- 底盘中心离地 = 轮半径 + 少量底盘厚度余量 -->
-    <origin xyz="0 0 ${wheel_radius}" rpy="0 0 0"/>
+    <!-- 底盘几何中心离地高度 = 轮半径 + 底盘高度/2。
+         这样底盘底面恰好位于轮子中心高度（z=wheel_radius），
+         轮子从底盘底面伸出接触地面，而不会埋在地下或浮在半空。 -->
+    <origin xyz="0 0 ${base_height/2 + wheel_radius}" rpy="0 0 0"/>
   </joint>
   <!-- ================= 轮子宏 ================= -->
@@ -103,5 +106,8 @@
       <parent link="base_link"/>
       <child link="${prefix}_wheel_link"/>
-      <origin xyz="${x_sign*wheelbase/2.0} ${y_sign*track_width/2.0} 0"
+      <!-- 轮关节 Z = -base_height/2，使轮子中心位于底盘底面（base_link
+           原点是底盘几何中心，向下偏移半个底盘高度即到底面）。
+           配合 base_footprint_joint 的 Z 偏移，轮子底部恰好着地。 -->
+      <origin xyz="${x_sign*wheelbase/2.0} ${y_sign*track_width/2.0} ${-base_height/2}"
               rpy="0 0 0"/>
       <axis xyz="0 1 0"/>

Commit message: fix(smartcar_bringup): 同步 description 包的车身轴距与轮距几何参数

File: src/smartcar_bringup/urdf/smartcar.urdf.xacro (robot description, xacro)
@@ -23,12 +23,9 @@
   <xacro:arg name="serial_port" default="/dev/ttyUSB0"/>
   <xacro:arg name="baud_rate" default="115200"/>
-  <!-- ===== 几何常量（单位 m，2026-07-20 实车测量回填）===== -->
-  <!-- 底盘外形：长 220 mm × 宽 192 mm × 高 145 mm；麦轮 Ø60 mm、厚 30 mm。
-       轴距/轮距暂按底盘长宽近似（轮心距未单独卷尺时）；改此处时必须同步
-       controllers.yaml 的 sum_of_robot_center_projection_on_X_Y_axis。 -->
+  <!-- ===== 几何常量（单位 m，2026-07-22 从 smartcar_description 同步）===== -->
   <xacro:property name="wheel_radius" value="0.03"/>   <!-- 麦轮 Ø60mm → r=0.03 -->
-  <xacro:property name="wheel_width" value="0.03"/>    <!-- 轮厚 30 mm，仅可视化 -->
-  <xacro:property name="wheelbase" value="0.220"/>     <!-- 前后轴距 ≈ 底盘长 -->
-  <xacro:property name="track_width" value="0.192"/>   <!-- 左右轮距 ≈ 底盘宽 -->
+  <xacro:property name="wheel_width" value="0.03062"/> <!-- 轮厚 30.62 mm -->
+  <xacro:property name="wheelbase" value="0.135"/>     <!-- 前后轴距 135 mm (CAD 精确轴距) -->
+  <xacro:property name="track_width" value="0.16462"/> <!-- 左右轮距 164.62 mm (CAD 精确轮距) -->
   <xacro:property name="base_length" value="0.220"/>
   <xacro:property name="base_width" value="0.192"/>
